File: Circuito/schematic.brd (EAGLE design)
At the start: 183.2 x 117 mm, 37 parts, among them IC2 7805TV

Commit message: Add files via upload
Parts:
- moved D18 27.9 mm to (15.2, 68.3)
- moved D10 27.9 mm to (15.0, 45.1)
- moved D11 27.9 mm to (32.0, 36.2)
- moved D12 27.9 mm to (34.7, 36.2)
- moved D23 27.9 mm to (15.0, 52.5)
- moved D7 27.9 mm to (15.0, 4.32)
- moved U$3 27.9 mm to (35.3, 61.7)
- moved U$4 27.9 mm to (49.3, 4.32)
- moved X3 27.9 mm to (5.47, 62.6)
- moved D1 27.9 mm to (15.4, 23.1)
- moved D15 27.9 mm to (15.0, 28.6)
- moved D16 27.9 mm to (15.0, 32.0)
- moved D5 27.9 mm to (23.1, 9.40)
- moved D6 27.9 mm to (25.6, 9.40)
- moved C1 27.9 mm to (47.5, 75.5)
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Routing:
- net N$16: track 0.00 -> 84.3 mm
- net N$14: track 0.00 -> 84.3 mm
- net N$19: track 0.00 -> 68.3 mm
- net N$15: track 0.00 -> 68.3 mm
Other:
- board size 183.2 x 117 mm -> 68.3 x 84.3 mm
